File: PCB/Slave/Slave.kicad_pcb (KiCad board)
At the start: 2 copper layers, 54.1 x 45.5 mm, 74 parts, among them J1 USB_C_Receptacle_USB2.0_16P, J2 Conn_01x05_Pin, J3 Conn_01x07_Socket, J4 Conn_01x04_Socket, J5 Conn_01x07_Socket, Q2 PNP, SW1 PTS810_SJM_250_SMTR_LFS, SW2 PTS810_SJM_250_SMTR_LFS, U1 ESP32-S3-MINI-1, U2 TCA9406DC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

Commit message: V3
Parts:
- removed the ? at (30.8, 58.4)
- removed the ? at (30.8, 56.1)
- removed the ? at (30.8, 56.9)
- removed the ? at (32.3, 56.1)
- removed the ? at (30.8, 57.6)
- removed the ? at (32.3, 57.6)
- removed the ? at (32.3, 56.9)
- removed the ? at (32.3, 58.4)
- added ?: , , F.Cu at (30.8, 56.9)
- added ?: , , F.Cu at (32.2, 58.4)
- added ?: , , F.Cu at (32.2, 56.1)
- added ?: , , F.Cu at (30.8, 57.6)
- added ?: , , F.Cu at (30.8, 58.4)
- added ?: , , F.Cu at (32.2, 57.6)
- added ?: , , F.Cu at (30.8, 56.1)
- added ?: , , F.Cu at (32.2, 56.9)
- added G***: LOGO, LOGO, B.Cu at (71.8, 45.2)
- moved C5 0.39 mm to (24.2, 57.5)
- moved C6 0.39 mm to (22.7, 57.5)
- moved C8 0.39 mm to (23.4, 53.5)
- moved U7 0.39 mm to (27.3, 53.3)
- moved C7 0.39 mm to (25.0, 53.5)
- moved J5 0.39 mm to (26.0, 61.6)
- moved MK1 0.39 mm to (27.0, 57.1)
- moved H2 0.16 mm to (26.0, 49.1)
Routing:
- net VCC_5V: track 131.7 -> 119.1 mm
- net I2S_SD: track 27.2 -> 26.3 mm
- net I2C_SCL_LINE: track 9.77 -> 10.3 mm
- net GND_OUT: track 116.4 -> 116.0 mm, vias 93 -> 92
Other:
- board size 54.1 x 45.5 mm -> 54.5 x 45 mm
- board text added: "E+"
- board text added: "E-"
- board text added: "MIC"
- board text added: "SLAVE PROBE V3"
- board text added: "SMART HIVE SLAVE V3"

Commit message: Update_Prosinec
Parts:
- removed ? (x8): , 
- U1: footprint RF_Module:ESP32-S2-MINI-1 -> ESP32-S3-MINI-1-N8:XCVR_ESP32-S3-MINI-1-N8
- moved U1 2.56 mm to (65.3, 51.1)
